Commit message: 修正驱动轮位置，消除行驶中"翘头"导致的雷达扫地
现象：机器人一前进就以前轮轴为支点抬起，俯仰稳定在 -7.238°，
激光雷达随之俯仰，360 束里有 164 束打到地面。

定位（用 Gazebo 的真实位姿 /world/default/pose/*，不是 /odom）：
- 静止俯仰 0.000°，一前进就变成 -7.238° 并保持不变，倒车则全程 0.000°。
- 该角度是几何硬约束：底盘后下棱相对轮轴为 (-0.2, -0.025)，
  0.2*sin(b) - 0.025*cos(b) = -0.05 的唯一解是 b = -7.2362°，
  与实测 -7.238° 相差 0.002° —— 机器人正是以后底盘棱为支点停住。
- 原因是重心几乎正压在驱动轮轴上（x_com ≈ +5 mm），
  翘头所需力矩仅 m*g*x_com ≈ 0.3 N·m，而巡航本身就要这么多；
  抬到 7.24° 后重心恰好落到轮轴正上方，于是稳定地停在这个姿态。
- 倒车时前侧万向轮本来就着地，顶住了下俯，所以看不到对称现象。

修改：wheel_offset_x 由 0.0 改为 -0.08，把轮轴后移 8cm，
恢复力矩升到约 5.2 N·m。

验证（重跑前进 1.8m）：
  俯仰           -7.238° -> 0.000°
  地面回波束数   164/帧  -> 0/帧
  墙面回波误差   mean 9mm（等于配置的高斯噪声 stddev=0.01）
  pitch/roll/z   0.000° / 0.000° / 0.1000m 全程不变

File: src/my_robot_description/urdf/my_robot.urdf.xacro (robot description, xacro)
@@ -7,5 +7,12 @@
   <xacro:property name="wheel_radius" value="0.05"/>
   <xacro:property name="wheel_width"  value="0.03"/>
-  <xacro:property name="wheel_offset_x" value="0.0"/>
+  <!-- 驱动轮轴必须明显位于重心之后，否则驱动力矩的反作用会让机器人"翘头"。
+       原先 wheel_offset_x=0.0，重心几乎正压在轮轴上，翘头所需的力矩只有
+       m*g*x_com ≈ 6.3*9.8*0.005 ≈ 0.3 N·m，而巡航本身需要的力矩就有这个量级，
+       于是机器人一路以前轮轴为支点抬到后底盘棱触地（正好 7.236°，见
+       laser_joint 偏置与底盘尺寸），并且重心此时恰好落到轮轴正上方而保持不倒。
+       后果是激光雷达随之俯仰 7.24°，把地面扫了进来（360 束里有 164 束打到地面）。
+       把轮轴后移 0.08 m 后，恢复力矩升到约 5.2 N·m，翘头不再发生。 -->
+  <xacro:property name="wheel_offset_x" value="-0.08"/>
   <xacro:property name="wheel_offset_y" value="0.17"/>
   <xacro:property name="wheel_offset_z" value="-0.05"/>

Commit message: 加后万向轮顶住翘头，兼顾里程计精度
上一步把驱动轮后移 0.08m 虽消除了翘头，但重心随之前移，
前万向轮开始承受约 31% 重量；原地旋转时这个固定球体只能拖地滑行，
轮子实际转速远超车体转角，里程计角速度虚高：
    odom wz = 0.8000 rad/s（恰等于指令值）
    true wz = 0.4900 rad/s
    => 1.679 倍

改为轮轴保持在底盘中心（重心仍压在轴线上，两个万向轮几乎不受力），
另在车尾 x=-0.15 增加一个等高的万向轮。抬头旋转会立刻被地面顶住，
绕后支点的恢复力矩由 0.3 N·m 升到约 9.6 N·m。

注：万向轮是 fixed joint，URDF->SDF 时会并入 base_link，
因此没法用 <gazebo reference="caster_wheel"> 单独设摩擦
（生成的 SDF 里是 base_link_fixed_joint_lump__caster_wheel_collision_1）。
所以这里靠几何而不是靠摩擦参数解决。

验证（同一次运行内先前进 1.8m 再原地旋转 8s）：
  前进段   pitch -0.003..0.000 deg，地面回波 0 帧，墙面误差 9.1mm
  旋转段   odom wz 0.8000 / true wz 0.7971 => 比值 1.011（改前 1.823）
  整段     pitch -0.009..0.002 deg
启动自检：/scan 9.771 Hz，静止位姿 (0,0,0.100) 且 RPY 全零。

File: src/my_robot_description/urdf/my_robot.urdf.xacro (robot description, xacro)
@@ -7,12 +7,13 @@
   <xacro:property name="wheel_radius" value="0.05"/>
   <xacro:property name="wheel_width"  value="0.03"/>
-  <!-- 驱动轮轴必须明显位于重心之后，否则驱动力矩的反作用会让机器人"翘头"。
-       原先 wheel_offset_x=0.0，重心几乎正压在轮轴上，翘头所需的力矩只有
-       m*g*x_com ≈ 6.3*9.8*0.005 ≈ 0.3 N·m，而巡航本身需要的力矩就有这个量级，
-       于是机器人一路以前轮轴为支点抬到后底盘棱触地（正好 7.236°，见
-       laser_joint 偏置与底盘尺寸），并且重心此时恰好落到轮轴正上方而保持不倒。
-       后果是激光雷达随之俯仰 7.24°，把地面扫了进来（360 束里有 164 束打到地面）。
-       把轮轴后移 0.08 m 后，恢复力矩升到约 5.2 N·m，翘头不再发生。 -->
-  <xacro:property name="wheel_offset_x" value="-0.08"/>
+  <!-- 轮轴保持在底盘中心。重心 x_com≈+5mm 几乎正压在轮轴上：翘头所需力矩只有
+       m*g*x_com ≈ 0.3 N·m，而巡航本身就要这么多，于是驱动力矩的反作用会把车
+       以前轮轴为支点抬起来，直到后底盘棱触地（几何上正好 7.236°，实测 -7.238°），
+       此时重心恰好落到轮轴正上方而停住。雷达随之俯仰 7.24°，把地面扫进来
+       （360 束里 164 束打到地面）。
+       试过把轮轴后移 0.08m：翘头没了，但重心前移使前万向轮承受约 31% 重量，
+       原地旋转时这个固定球体拖地打滑，里程计角速度虚高 1.68 倍（实测 0.8 vs 0.49）。
+       因此改为轮轴居中，另加一个后万向轮从几何上顶住翘头。 -->
+  <xacro:property name="wheel_offset_x" value="0.0"/>
   <xacro:property name="wheel_offset_y" value="0.17"/>
   <xacro:property name="wheel_offset_z" value="-0.05"/>
@@ -128,4 +129,36 @@
     <child link="caster_wheel"/>
     <origin xyz="0.15 0 -0.08" rpy="0 0 0"/>
+  </joint>
+  <!-- ========== 后万向轮 ==========
+       只起"防翘头"作用：重心几乎压在驱动轮轴上，向后转的恢复力矩很小，
+       驱动力矩的反作用会让车头抬起。后方多一个等高支点后，抬头的旋转立刻
+       被地面顶住（绕后支点的恢复力矩升到约 9.6 N·m）。
+       它与前万向轮一样几乎不受力，所以不会像"轮轴后移"那样给原地旋转
+       带来拖地打滑。 -->
+  <link name="rear_caster">
+    <visual>
+      <geometry>
+        <sphere radius="${caster_radius}"/>
+      </geometry>
+      <material name="gray">
+        <color rgba="0.5 0.5 0.5 1.0"/>
+      </material>
+    </visual>
+    <collision>
+      <geometry>
+        <sphere radius="${caster_radius}"/>
+      </geometry>
+    </collision>
+    <inertial>
+      <mass value="0.2"/>
+      <inertia ixx="0.0001" ixy="0" ixz="0"
+               iyy="0.0001" iyz="0"
+               izz="0.0001"/>
+    </inertial>
+  </link>
+  <joint name="rear_caster_joint" type="fixed">
+    <parent link="base_link"/>
+    <child link="rear_caster"/>
+    <origin xyz="-0.15 0 -0.08" rpy="0 0 0"/>
   </joint>
   <!-- ========== 激光雷达 ========== -->

Commit message: 按实车改为四轮全驱 skid-steer
实车是四个轮子（左右各两个、全驱），之前的两轮+万向轮模型不对。
本次把 URDF 重建为 skid-steer，并删掉此前为绕开翘头而加的前后万向轮
（207fe13/7632380 那两版的结论仍然有效，但补丁本身已不需要）。

顺带查出一个一直存在的死配置：
  max_wheel_torque / max_wheel_acceleration 这两个参数在 gz-sim 8.15.0 的
  DiffDrive 里根本不存在——官方文档（v8 和 v9）都没有，二进制里也搜不到，
  两条独立证据一致。也就是说驱动力矩一直是**无上限**的。
  真正认的是 max_velocity / max_acceleration / max_jerk 及其分轴版本，
  已改用 max_linear/angular_velocity 和 max_linear/angular_acceleration。

几何（0.4x0.3 底盘，占位值，待按实车实测修改）：
  轴距 0.28（wheel_offset_x=0.14），轮距 0.34，轮半径 0.05，轮宽 0.03
  整机 6.5 kg，重心在中心，支撑多边形 x∈[-0.14,0.14] y∈[-0.17,0.17]
  翘头恢复力矩 m*g*0.14 ≈ 8.9 N·m（旧结构只有 0.3 N·m）

skid-steer 的关键取舍：四轮平行，原地转必然横向刮擦，编码器里程计
必然虚高。这是实车固有特性，因此**保留**而不是消除。
用摩擦各向异性建模（mu=1.0 纵向 / mu2=0.5 横向，fdir1=1 0 0），
mu2 就是"打滑程度"的标定旋钮。

实测（前进 0.3m/s 6s + 原地旋转 0.8rad/s 8s）：
  俯仰/横滚           +-0.003 deg（无翘头）
  前进段地面回波      0/20 帧
  前进段墙面误差      9.2 mm（配置噪声 stddev=10mm）
  前进段里程计 x 误差 平均 -4.1mm，最大 6.6mm
  直线度              y 漂移 0.0mm，yaw 漂移 0.000 deg
  静止基线            83 束命中 / 276 束 inf 一致，与改动前完全一致
  旋转段 odom/true    1.380（中位 1.394）<- skid-steer 真实打滑

运行时实体树确认 5 个 link：base_link + 四个轮子。

File: src/my_robot_description/urdf/my_robot.urdf.xacro (robot description, xacro)
@@ -1,22 +1,89 @@
 <?xml version="1.0"?>
 <robot xmlns:xacro="http://www.ros.org/wiki/xacro" name="my_robot">
-  <!-- ========== 参数定义 ========== -->
-  <xacro:property name="base_length" value="0.4"/>
-  <xacro:property name="base_width"  value="0.3"/>
-  <xacro:property name="base_height" value="0.15"/>
+  <!-- ================================================================
+       四轮全驱 skid-steer（按实车建）
+       ================================================================
+       左右各两个驱动轮，全部由 DiffDrive 驱动，没有万向轮。
+       为什么这样能同时解决之前两个问题：
+       1) 翘头：支撑多边形在 x 方向横跨前后轴（±wheel_offset_x），
+          抬头要绕后轴翻转，恢复力矩 m*g*wheel_offset_x ≈ 8.9 N·m，
+          而之前两轮+万向轮时只有 0.3 N·m，所以再也不会翘。
+          雷达不俯仰，自然也不会扫到地面。
+       2) 原地旋转的里程计误差：四轮平行，原地转时每个轮子都必须
+          横向刮擦，编码器积分出来的转角必然与车体真实转角不符。
+          这是 skid-steer 的固有特性，实车同样存在，所以这里**保留**
+          而不是消除——让上层的 SLAM/Nav2 面对和实车一样的里程计质量。
+       ★ 下面 7 个几何/质量/限速参数是按 0.4×0.3 底盘估的占位值，
+         请按实车实测值修改（尤其 wheel_offset_x = 半轴距）。
+       ================================================================ -->
+  <xacro:property name="base_length"  value="0.4"/>
+  <xacro:property name="base_width"   value="0.3"/>
+  <xacro:property name="base_height"  value="0.15"/>
+  <xacro:property name="base_mass"    value="5.0"/>
   <xacro:property name="wheel_radius" value="0.05"/>
   <xacro:property name="wheel_width"  value="0.03"/>
-  <!-- 轮轴保持在底盘中心。重心 x_com≈+5mm 几乎正压在轮轴上：翘头所需力矩只有
-       m*g*x_com ≈ 0.3 N·m，而巡航本身就要这么多，于是驱动力矩的反作用会把车
-       以前轮轴为支点抬起来，直到后底盘棱触地（几何上正好 7.236°，实测 -7.238°），
-       此时重心恰好落到轮轴正上方而停住。雷达随之俯仰 7.24°，把地面扫进来
-       （360 束里 164 束打到地面）。
-       试过把轮轴后移 0.08m：翘头没了，但重心前移使前万向轮承受约 31% 重量，
-       原地旋转时这个固定球体拖地打滑，里程计角速度虚高 1.68 倍（实测 0.8 vs 0.49）。
-       因此改为轮轴居中，另加一个后万向轮从几何上顶住翘头。 -->
-  <xacro:property name="wheel_offset_x" value="0.0"/>
-  <xacro:property name="wheel_offset_y" value="0.17"/>
+  <xacro:property name="wheel_mass"   value="0.35"/>
+  <xacro:property name="wheel_offset_x" value="0.14"/>  <!-- 半轴距，实车轴距 = 0.28 -->
+  <xacro:property name="wheel_offset_y" value="0.17"/>  <!-- 半轮距，实车轮距 = 0.34 -->
   <xacro:property name="wheel_offset_z" value="-0.05"/>
-  <xacro:property name="caster_radius" value="0.02"/>
+  <!-- skid-steer 的摩擦各向异性。
+       真实轮子横向阻力比纵向小得多（胎面/接触面变形），这个比值直接决定
+       原地旋转时打滑多少。先用 1.0 / 0.5 起步，实测出来的 odom/true 比值
+       要和实车对比后再调——真实值只能靠实车标定。 -->
+  <xacro:property name="wheel_mu_long" value="1.0"/>   <!-- 沿滚动方向 -->
+  <xacro:property name="wheel_mu_lat"  value="0.5"/>   <!-- 垂直滚动方向 -->
+  <!-- ★ 速度/加速度上限：实车实测值待填。
+       注意这些才是 gz-sim 8 真正认的参数；之前 URDF 里的
+       max_wheel_torque / max_wheel_acceleration 在 8.15.0 的 DiffDrive
+       文档和二进制里都不存在，写了也从来没生效过。 -->
+  <xacro:property name="max_linear_vel"  value="0.5"/>
+  <xacro:property name="max_angular_vel" value="1.5"/>
+  <xacro:property name="max_linear_acc"  value="0.5"/>
+  <xacro:property name="max_angular_acc" value="2.0"/>
+  <!-- ========== 驱动轮宏 ========== -->
+  <xacro:macro name="drive_wheel" params="name x y">
+    <link name="${name}">
+      <visual>
+        <geometry>
+          <cylinder radius="${wheel_radius}" length="${wheel_width}"/>
+        </geometry>
+        <origin xyz="0 0 0" rpy="1.5708 0 0"/>
+        <material name="black">
+          <color rgba="0.1 0.1 0.1 1.0"/>
+        </material>
+      </visual>
+      <collision>
+        <geometry>
+          <cylinder radius="${wheel_radius}" length="${wheel_width}"/>
+        </geometry>
+        <origin xyz="0 0 0" rpy="1.5708 0 0"/>
+      </collision>
+      <inertial>
+        <mass value="${wheel_mass}"/>
+        <inertia ixx="0.0005" ixy="0" ixz="0"
+                 iyy="0.0005" iyz="0"
+                 izz="0.0005"/>
+      </inertial>
+    </link>
+    <joint name="${name}_joint" type="continuous">
+      <parent link="base_link"/>
+      <child link="${name}"/>
+      <origin xyz="${x} ${y} ${wheel_offset_z}" rpy="0 0 0"/>
+      <axis xyz="0 1 0"/>
+    </joint>
+    <!-- fdir1 在碰撞体坐标系里表达；碰撞体只绕 x 转了 90°，
+         所以 x 轴不变，fdir1=1 0 0 就是轮子的滚动方向。 -->
+    <gazebo reference="${name}">
+      <surface>
+        <friction>
+          <ode>
+            <mu>${wheel_mu_long}</mu>
+            <mu2>${wheel_mu_lat}</mu2>
+            <fdir1>1 0 0</fdir1>
+          </ode>
+        </friction>
+      </surface>
+    </gazebo>
+  </xacro:macro>
   <!-- ========== 底盘 ========== -->
   <link name="base_link">
@@ -37,5 +104,5 @@
     </collision>
     <inertial>
-      <mass value="5.0"/>
+      <mass value="${base_mass}"/>
       <inertia ixx="0.05" ixy="0" ixz="0"
                iyy="0.08" iyz="0"
@@ -43,123 +110,9 @@
     </inertial>
   </link>
-  <!-- ========== 左驱动轮 ========== -->
-  <link name="left_wheel">
-    <visual>
-      <geometry>
-        <cylinder radius="${wheel_radius}" length="${wheel_width}"/>
-      </geometry>
-      <origin xyz="0 0 0" rpy="1.5708 0 0"/>
-      <material name="black">
-        <color rgba="0.1 0.1 0.1 1.0"/>
-      </material>
-    </visual>
-    <collision>
-      <geometry>
-        <cylinder radius="${wheel_radius}" length="${wheel_width}"/>
-      </geometry>
-      <origin xyz="0 0 0" rpy="1.5708 0 0"/>
-    </collision>
-    <inertial>
-      <mass value="0.5"/>
-      <inertia ixx="0.001" ixy="0" ixz="0"
-               iyy="0.001" iyz="0"
-               izz="0.001"/>
-    </inertial>
-  </link>
-  <joint name="left_wheel_joint" type="continuous">
-    <parent link="base_link"/>
-    <child link="left_wheel"/>
-    <origin xyz="${wheel_offset_x} ${wheel_offset_y} ${wheel_offset_z}" rpy="0 0 0"/>
-    <axis xyz="0 1 0"/>
-  </joint>
-  <!-- ========== 右驱动轮 ========== -->
-  <link name="right_wheel">
-    <visual>
-      <geometry>
-        <cylinder radius="${wheel_radius}" length="${wheel_width}"/>
-      </geometry>
-      <origin xyz="0 0 0" rpy="1.5708 0 0"/>
-      <material name="black">
-        <color rgba="0.1 0.1 0.1 1.0"/>
-      </material>
-    </visual>
-    <collision>
-      <geometry>
-        <cylinder radius="${wheel_radius}" length="${wheel_width}"/>
-      </geometry>
-      <origin xyz="0 0 0" rpy="1.5708 0 0"/>
-    </collision>
-    <inertial>
-      <mass value="0.5"/>
-      <inertia ixx="0.001" ixy="0" ixz="0"
-               iyy="0.001" iyz="0"
-               izz="0.001"/>
-    </inertial>
-  </link>
-  <joint name="right_wheel_joint" type="continuous">
-    <parent link="base_link"/>
-    <child link="right_wheel"/>
-    <origin xyz="${wheel_offset_x} -${wheel_offset_y} ${wheel_offset_z}" rpy="0 0 0"/>
-    <axis xyz="0 1 0"/>
-  </joint>
-  <!-- ========== 万向轮 ========== -->
-  <link name="caster_wheel">
-    <visual>
-      <geometry>
-        <sphere radius="${caster_radius}"/>
-      </geometry>
-      <material name="gray">
-        <color rgba="0.5 0.5 0.5 1.0"/>
-      </material>
-    </visual>
-    <collision>
-      <geometry>
-        <sphere radius="${caster_radius}"/>
-      </geometry>
-    </collision>
-    <inertial>
-      <mass value="0.2"/>
-      <inertia ixx="0.0001" ixy="0" ixz="0"
-               iyy="0.0001" iyz="0"
-               izz="0.0001"/>
-    </inertial>
-  </link>
-  <joint name="caster_joint" type="fixed">
-    <parent link="base_link"/>
-    <child link="caster_wheel"/>
-    <origin xyz="0.15 0 -0.08" rpy="0 0 0"/>
-  </joint>
-  <!-- ========== 后万向轮 ==========
-       只起"防翘头"作用：重心几乎压在驱动轮轴上，向后转的恢复力矩很小，
-       驱动力矩的反作用会让车头抬起。后方多一个等高支点后，抬头的旋转立刻
-       被地面顶住（绕后支点的恢复力矩升到约 9.6 N·m）。
-       它与前万向轮一样几乎不受力，所以不会像"轮轴后移"那样给原地旋转
-       带来拖地打滑。 -->
-  <link name="rear_caster">
-    <visual>
-      <geometry>
-        <sphere radius="${caster_radius}"/>
-      </geometry>
-      <material name="gray">
-        <color rgba="0.5 0.5 0.5 1.0"/>
-      </material>
-    </visual>
-    <collision>
-      <geometry>
-        <sphere radius="${caster_radius}"/>
-      </geometry>
-    </collision>
-    <inertial>
-      <mass value="0.2"/>
-      <inertia ixx="0.0001" ixy="0" ixz="0"
-               iyy="0.0001" iyz="0"
-               izz="0.0001"/>
-    </inertial>
-  </link>
-  <joint name="rear_caster_joint" type="fixed">
-    <parent link="base_link"/>
-    <child link="rear_caster"/>
-    <origin xyz="-0.15 0 -0.08" rpy="0 0 0"/>
-  </joint>
+  <!-- ========== 四个驱动轮 ========== -->
+  <xacro:drive_wheel name="front_left_wheel"  x="${wheel_offset_x}"  y="${wheel_offset_y}"/>
+  <xacro:drive_wheel name="rear_left_wheel"   x="-${wheel_offset_x}" y="${wheel_offset_y}"/>
+  <xacro:drive_wheel name="front_right_wheel" x="${wheel_offset_x}"  y="-${wheel_offset_y}"/>
+  <xacro:drive_wheel name="rear_right_wheel"  x="-${wheel_offset_x}" y="-${wheel_offset_y}"/>
   <!-- ========== 激光雷达 ========== -->
   <link name="laser_frame">
@@ -189,13 +142,17 @@
     <origin xyz="0.0 0 0.12" rpy="0 0 0"/>
   </joint>
-    <!-- ========== Gazebo 差速驱动插件 ========== -->
+  <!-- ========== Gazebo 差速驱动插件 ==========
+       一侧挂两个 joint 是官方支持的：文档明确写
+       "can be attached to a model with any number of left and right wheels"，
+       且 <left_joint>/<right_joint> "can appear multiple times"。
+       wheel_separation 仍然是左右轮距（0.34），与轴距无关。 -->
   <gazebo>
     <plugin filename="gz-sim-diff-drive-system" name="gz::sim::systems::DiffDrive">
-      <left_joint>left_wheel_joint</left_joint>
-      <right_joint>right_wheel_joint</right_joint>
-      <wheel_separation>0.34</wheel_separation>
-      <wheel_radius>0.05</wheel_radius>
-      <max_wheel_torque>20</max_wheel_torque>
-      <max_wheel_acceleration>1.0</max_wheel_acceleration>
+      <left_joint>front_left_wheel_joint</left_joint>
+      <left_joint>rear_left_wheel_joint</left_joint>
+      <right_joint>front_right_wheel_joint</right_joint>
+      <right_joint>rear_right_wheel_joint</right_joint>
+      <wheel_separation>${2 * wheel_offset_y}</wheel_separation>
+      <wheel_radius>${wheel_radius}</wheel_radius>
       <odom_topic>odom</odom_topic>
       <tf_topic>tf</tf_topic>
@@ -203,4 +160,9 @@
       <child_frame_id>base_link</child_frame_id>
       <topic>cmd_vel</topic>
+      <odom_publish_frequency>50</odom_publish_frequency>
+      <max_linear_velocity>${max_linear_vel}</max_linear_velocity>
+      <max_angular_velocity>${max_angular_vel}</max_angular_velocity>
+      <max_linear_acceleration>${max_linear_acc}</max_linear_acceleration>
+      <max_angular_acceleration>${max_angular_acc}</max_angular_acceleration>
     </plugin>
   </gazebo>

Commit message: 把雷达参数提成 xacro property，集中实车待测值并加清单文档

File: src/my_robot_description/urdf/my_robot.urdf.xacro (robot description, xacro)
@@ -14,6 +14,12 @@
           这是 skid-steer 的固有特性，实车同样存在，所以这里**保留**
           而不是消除——让上层的 SLAM/Nav2 面对和实车一样的里程计质量。
-       ★ 下面 7 个几何/质量/限速参数是按 0.4×0.3 底盘估的占位值，
-         请按实车实测值修改（尤其 wheel_offset_x = 半轴距）。
+       ★★ 下面这一段 property 是本工程**唯一**依赖实车实测数据的地方。
+          全部是按 0.4×0.3 底盘估的占位值，不是实测值。
+          拿到实车数据后怎么改：
+            1. 只改这一段（几何 / 质量 / 限速 / 摩擦 / 雷达，共 5 组）；
+            2. 不用 colcon build —— install 是符号链接，直接指向本文件；
+            3. 重启 launch 即可生效。
+          改哪个值要连带改哪里（Nav2、SLAM），见 docs/real_robot_params.md。
+          最要紧的是 wheel_offset_x（半轴距）和雷达安装高度 / 量程。
        ================================================================ -->
   <xacro:property name="base_length"  value="0.4"/>
@@ -41,4 +47,17 @@
   <xacro:property name="max_linear_acc"  value="0.5"/>
   <xacro:property name="max_angular_acc" value="2.0"/>
+  <!-- ★ 雷达参数：同样是占位值，从未和实车雷达核对过。
+       雷达装高一点（比如 0.25）能少扫到地面；量程和角度要按实车型号改，
+       否则 SLAM 会把真实存在的墙当成"超出量程"而丢掉。 -->
+  <xacro:property name="lidar_mount_x"  value="0.0"/>    <!-- 相对 base_link -->
+  <xacro:property name="lidar_mount_y"  value="0.0"/>
+  <xacro:property name="lidar_mount_z"  value="0.12"/>
+  <xacro:property name="lidar_samples"  value="360"/>    <!-- 水平线数 -->
+  <xacro:property name="lidar_min_angle" value="-3.14159"/>
+  <xacro:property name="lidar_max_angle" value="3.14159"/>
+  <xacro:property name="lidar_range_min" value="0.1"/>
+  <xacro:property name="lidar_range_max" value="12.0"/>
+  <xacro:property name="lidar_update_rate" value="10"/>  <!-- Hz -->
+  <xacro:property name="lidar_noise_stddev" value="0.01"/> <!-- m -->
   <!-- ========== 驱动轮宏 ========== -->
   <xacro:macro name="drive_wheel" params="name x y">
@@ -140,5 +159,5 @@
     <parent link="base_link"/>
     <child link="laser_frame"/>
-    <origin xyz="0.0 0 0.12" rpy="0 0 0"/>
+    <origin xyz="${lidar_mount_x} ${lidar_mount_y} ${lidar_mount_z}" rpy="0 0 0"/>
   </joint>
   <!-- ========== Gazebo 差速驱动插件 ==========
@@ -172,5 +191,5 @@
       <always_on>true</always_on>
       <visualize>true</visualize>
-      <update_rate>10</update_rate>
+      <update_rate>${lidar_update_rate}</update_rate>
       <topic>scan</topic>
       <gz_frame_id>laser_frame</gz_frame_id>
@@ -178,17 +197,17 @@
         <scan>
           <horizontal>
-            <samples>360</samples>
-            <min_angle>-3.14159</min_angle>
-            <max_angle>3.14159</max_angle>
+            <samples>${lidar_samples}</samples>
+            <min_angle>${lidar_min_angle}</min_angle>
+            <max_angle>${lidar_max_angle}</max_angle>
           </horizontal>
         </scan>
         <range>
-          <min>0.1</min>
-          <max>12.0</max>
+          <min>${lidar_range_min}</min>
+          <max>${lidar_range_max}</max>
         </range>
         <noise>
           <type>gaussian</type>
           <mean>0.0</mean>
-          <stddev>0.01</stddev>
+          <stddev>${lidar_noise_stddev}</stddev>
         </noise>
       </lidar>

Commit message: 标定 skid-steer 有效轮距：wheel_separation_scale = 1.36
四轮 skid-steer 原地转时轮子横向刮擦，DiffDrive 用几何轮距 0.34 m
同时算"指令→轮速差"和"轮速差→里程计"，于是一个倍率污染两件事：

    odom/真值 = 1.36   （里程计报的转角比真实大 36%）
    真值/指令 = 0.73   （命令转 1 圈，实际只转 0.73 圈）

解法是把插件的 wheel_separation 换成有效轮距 b·scale：

    指令侧 Δv = ω_cmd·b_eff  →  ω_true = ω_cmd          ✅
    里程计侧 ω_odom = Δv/b_eff = ω_true                  ✅

一个系数同时修好控制增益和里程计标度，而且不动物理（刮擦照旧）。

1.36 来自实测：原地转 ω=0.6/1.2/1.5 rad/s 四个工况，
odom/真值 = 1.355 / 1.355 / 1.364 / 1.361，标定后为
1.040 / 1.000 / 1.003。弧线工况标定后仍差 9%（侧滑量随曲率变化，
单一标量只能折中，优先照顾原地转）。

⚠ 这是仿真值，实车必须用同样方法重测后填入。

File: src/my_robot_description/urdf/my_robot.urdf.xacro (robot description, xacro)
@@ -12,10 +12,11 @@
        2) 原地旋转的里程计误差：四轮平行，原地转时每个轮子都必须
           横向刮擦，编码器积分出来的转角必然与车体真实转角不符。
-          这是 skid-steer 的固有特性，实车同样存在，所以这里**保留**
-          而不是消除——让上层的 SLAM/Nav2 面对和实车一样的里程计质量。
+          这是 skid-steer 的固有特性，实车同样存在，所以物理上**保留**
+          这个刮擦（不去"修正"摩擦系数把它磨平）。
+          但**上报**的里程计要标定：见下面的 wheel_separation_scale。
        ★★ 下面这一段 property 是本工程**唯一**依赖实车实测数据的地方。
           全部是按 0.4×0.3 底盘估的占位值，不是实测值。
           拿到实车数据后怎么改：
-            1. 只改这一段（几何 / 质量 / 限速 / 摩擦 / 雷达，共 5 组）；
+            1. 只改这一段（几何 / 质量 / 限速 / 摩擦 / 打滑标定 / 雷达，共 6 组）；
             2. 不用 colcon build —— install 是符号链接，直接指向本文件；
             3. 重启 launch 即可生效。
@@ -39,4 +40,26 @@
   <xacro:property name="wheel_mu_long" value="1.0"/>   <!-- 沿滚动方向 -->
   <xacro:property name="wheel_mu_lat"  value="0.5"/>   <!-- 垂直滚动方向 -->
+  <!-- ★★★ 有效轮距标定系数（skid-steer 最重要的一项标定）
+       问题：DiffDrive 插件用几何轮距 b=0.34 把角速度换算成左右轮速差
+             Δv = ω_b，再用同一个 b 反算里程计 ω_o = Δv/b。
+             但四轮侧滑让车体真实转角小于轮子"应该"转过的角度：
+                 ω_true = Δv / b_eff     其中 b_eff > b
+             于是 b_eff/b 这个倍率同时污染了**控制增益**和**里程计标度**：
+                 ω_o / ω_true = b_eff / b = 1.36
+                 ω_true / ω_cmd = b / b_eff = 0.73
+             即"命令转 1 圈，实际只转 0.73 圈，而里程计报 1 圈"。
+       解法：把插件里的 wheel_separation 换成 b_eff = b · 本系数。
+             指令侧 Δv = ω_cmd · b_eff →  ω_true = ω_cmd  ✅
+             里程计侧 ω_o = Δv / b_eff = ω_cmd = ω_true  ✅
+             一个系数同时修好两件事，且不需要动物理（刮擦照旧存在）。
+       1.36 的来源：本仓库实测（/tmp/step4/gains.py，原地转 ω=0.6/1.2/1.5
+       rad/s 三个工况），odom/真值 = 1.355 / 1.355 / 1.364 / 1.361。
+       数据与推导见 docs/nav2.md。
+       ⚠ 这个值必须用**实车**重测，方法是：原地以固定角速度转固定秒数，
+         比较"编码器积分出来的转角"和"实际转过的转角"（地上贴胶带/用
+         外部标定），比值填这里。仿真值与实车值不会一样。
+       ⚠ 转弯半径不同倍率也不同（侧滑量随曲率变化）。这里取原地转的值，
+         因为室内导航里原地转占绝大多数。弧线工况实测偏大约 5%，见 docs。 -->
+  <xacro:property name="wheel_separation_scale" value="1.36"/>
   <!-- ★ 速度/加速度上限：实车实测值待填。
        注意这些才是 gz-sim 8 真正认的参数；之前 URDF 里的
@@ -165,5 +188,7 @@
        "can be attached to a model with any number of left and right wheels"，
        且 <left_joint>/<right_joint> "can appear multiple times"。
-       wheel_separation 仍然是左右轮距（0.34），与轴距无关。 -->
+       wheel_separation 用的是**有效轮距** 2*wheel_offset_y*scale，
+       不是几何轮距 2*wheel_offset_y —— 原因见上面
+       wheel_separation_scale 的长注释。0.34 * 1.36 = 0.4624 m。 -->
   <gazebo>
     <plugin filename="gz-sim-diff-drive-system" name="gz::sim::systems::DiffDrive">
@@ -172,5 +197,5 @@
       <right_joint>front_right_wheel_joint</right_joint>
       <right_joint>rear_right_wheel_joint</right_joint>
-      <wheel_separation>${2 * wheel_offset_y}</wheel_separation>
+      <wheel_separation>${2 * wheel_offset_y * wheel_separation_scale}</wheel_separation>
       <wheel_radius>${wheel_radius}</wheel_radius>
       <odom_topic>odom</odom_topic>
